File: meteo_station/meteo_station.kicad_pcb (KiCad board)
At the start: 2 copper layers, 110 x 90 mm, 36 parts, among them SW1 SW_SPDT, U1 TP4056, U2 LF33_TO220, U3 ESP32-WROOM, U4 DS18B20, U5 BH1750, U6 BME280

Commit message: something
Parts:
- removed BT1: Battery, meteo_station_footprints:BatteryHolder
- removed C3, C5: 100nF, Capacitor_SMD:C_0603_1608Metric
- removed C4: 2.2uF, Capacitor_Tantalum_SMD:CP_EIA-3216-18_Kemet-A
- removed D1, D2: D_Schottky, Diode_SMD:D_SMB
- removed the G*** at (96.5, 130.0)
- removed JP1: SolderJumper, Jumper:SolderJumper-2_P1.3mm_Bridged_Pad1.0x1.5mm
- removed R3, R4, R5: 4.7K, Resistor_SMD:R_0603_1608Metric
- removed REF** (x4): MountingHole_3.2mm_M3, MountingHole:MountingHole_3.2mm_M3
- removed SC1, SC2: Solar_Cell, meteo_station_footprints:SolarPanel_JST
- removed SW1: SW_SPDT, meteo_station_footprints:MTS102
- removed U1: TP4056, meteo_station_footprints:TP4056
- removed U2: LF33_TO220, Package_TO_SOT_THT:TO-220-3_Horizontal_TabDown
- removed U4: DS18B20, meteo_station_footprints:TO-92_Inline
- removed U5: BH1750, meteo_station_footprints:BH1750
- added J2: PMS7003, Connector:NS-Tech_Grove_1x04_P2mm_Vertical, F.Cu at (106.7, 90.5)
- C2: footprint Capacitor_SMD:C_0603_1608Metric -> Capacitor_THT:C_Disc_D7.5mm_W2.5mm_P5.00mm
- R1, R2: footprint Resistor_SMD:R_0603_1608Metric -> Resistor_THT:R_Axial_DIN0207_L6.3mm_D2.5mm_P10.16mm_Horizontal
- moved G*** 170.7 mm to (325.1, -17.8)
- moved G*** 169.8 mm to (337.4, -2.79)
- moved U6 83.2 mm to (99.1, 113.0), turned to 180 degrees
- moved C2 59.7 mm to (109.2, 83.7), turned to 90 degrees
- moved R2 16.6 mm to (119.3, 88.9), turned to 90 degrees
- moved R1 16.4 mm to (116.8, 88.9)
- moved C1 8.75 mm to (126.1, 80.8), turned to 0 degrees
- moved U3 7.22 mm to (149.9, 100.3)
Connections:
- C2 pad 1: BAT_V -> ADC_BAT
- R1 pad 1: BAT_V -> ADC_BAT
- R1 pad 2: OUT+ -> 3V3
- R2 pad 1: BAT_V -> ADC_BAT
- R2 pad 2: OUT- -> GND
- U3 pad 15: unconnected-(U3-Pad15) -> 5V
- U3 pad 24: unconnected-(U3-Pad24) -> TX_PMS
- U3 pad 25: unconnected-(U3-Pad25) -> RX_PMS
- U3 pad 26: Net-(R5-Pad2) -> unconnected-(U3-D4-Pad26)
- U3 pad 4: BAT_V -> unconnected-(U3-D34-Pad4)
- U3 pad 7: unconnected-(U3-Pad7) -> ADC_BAT
Routing:
- net GND: track 0.00 -> 196.6 mm
- net Net-(R5-Pad2): track 100.3 -> 0.00 mm
- net Net-(BT1-Pad1): track 89.0 -> 0.00 mm
- net 3V3: track 164.9 -> 78.8 mm
- net ADC_BAT: track 0.00 -> 80.0 mm
- net SDA: track 106.3 -> 35.1 mm, vias 2 -> 0
- net BAT_V: track 67.6 -> 0.00 mm, vias 1 -> 0
- net Net-(D1-Pad1): track 65.5 -> 0.00 mm
- net SCL: track 88.7 -> 35.1 mm, vias 1 -> 0
- net Net-(BT1-Pad2): track 45.5 -> 0.00 mm
- net OUT+: track 33.8 -> 0.00 mm
- net TX_PMS: track 0.00 -> 31.5 mm
- net RX_PMS: track 0.00 -> 31.3 mm
- net Net-(SC1-Pad2): track 27.8 -> 0.00 mm
- net OUT-: track 17.6 -> 0.00 mm
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- removed copper zone on F.Cu, net GND
Other:
- board size 110 x 90 mm -> 255.9 x 148.1 mm
- board text removed: "3V3"

Commit message: something2
Parts:
- removed the G*** at (337.4, -2.79)
- removed the G*** at (325.1, -17.8)
- removed the G*** at (167.1, 76.2)
- removed the G*** at (133.3, 139.4)
- removed the G*** at (197.5, 151.6)
- removed the G*** at (149.9, 144.8)
- removed the G*** at (200.7, 100.3)
- removed the G*** at (101.2, 118.7)
- added G***: LOGO, meteo_station_footprints:chmurka2, F.Cu at (153.7, 115.6)
- added G***: LOGO, meteo_station_footprints:chmurka2, F.Cu at (108.0, 87.6)
- added M3: MountingHole_3mm, MountingHole:MountingHole_3mm, F.Cu at (161.4, 126.6)
- added M3: MountingHole_3mm, MountingHole:MountingHole_3mm, F.Cu at (102.8, 126.5)
- added REF**: MountingHole_3mm, MountingHole:MountingHole_3mm, F.Cu at (102.8, 76.9)
- C2: footprint Capacitor_THT:C_Disc_D7.5mm_W2.5mm_P5.00mm -> Capacitor_THT:C_Disc_D5.0mm_W2.5mm_P2.50mm
- J2: footprint Connector:NS-Tech_Grove_1x04_P2mm_Vertical -> Connector_PinHeader_2.54mm:PinHeader_1x04_P2.54mm_Horizontal
- moved C2 54.7 mm to (160.0, 104.1), turned to 135 degrees
- moved R1 46.2 mm to (161.3, 76.2), turned to -90 degrees
- moved R2 37.8 mm to (154.9, 76.2), turned to -90 degrees
- moved J2 34.4 mm to (110.2, 124.8), turned to 135 degrees
- moved C1 34.0 mm to (158.8, 90.2), turned to -90 degrees
- moved U6 18.8 mm to (110.6, 98.2), turned to 135 degrees
- moved U3 12.8 mm to (137.2, 101.6)
Connections:
- C1 pad 1: 3V3 -> 5V
Routing:
- net GND: track 196.6 -> 4.59 mm
- net 5V: track 0.00 -> 84.0 mm
- net ADC_BAT: track 80.0 -> 48.6 mm
- net SDA: track 35.1 -> 15.5 mm
- net RX_PMS: track 31.3 -> 48.6 mm
- net SCL: track 35.1 -> 22.2 mm
- net 3V3: track 78.8 -> 67.8 mm
- net TX_PMS: track 31.5 -> 39.8 mm
- added copper zone on F.Cu, net GND
- removed copper zone on B.Cu, net GND
Other:
- board size 255.9 x 148.1 mm -> 65.2 x 56.2 mm
- board text added: "Smoggy v1.0"
- board text removed: "alicja.space"
