File: meteo_station/meteo_station.kicad_sch (KiCad schematic)
At the start: 23 parts, among them SW1 SW_SPDT, U1 TP4056, U2 LF33_TO220, U3 ESP32-WROOM, U4 DS18B20, U5 BH1750, U6 BME280

Commit message: something
Parts:
- removed BT1: Battery, meteo_station_footprints:BatteryHolder, symbol Device:Battery
- removed C3, C5: 100nF, Capacitor_SMD:C_0603_1608Metric, symbol Device:C
- removed C4: 2.2uF, Capacitor_Tantalum_SMD:CP_EIA-3216-18_Kemet-A, symbol Device:C_Polarized_US
- removed D1, D2: D_Schottky, Diode_SMD:D_SMB, symbol Device:D_Schottky
- removed JP1: SolderJumper, Jumper:SolderJumper-2_P1.3mm_Bridged_Pad1.0x1.5mm, symbol Jumper:SolderJumper_2_Bridged
- removed R3, R4, R5: 4.7K, Resistor_SMD:R_0603_1608Metric, symbol Device:R
- removed SC1, SC2: Solar_Cell, meteo_station_footprints:SolarPanel_JST, symbol Device:Solar_Cell
- removed SW1: SW_SPDT, meteo_station_footprints:MTS102, symbol Switch:SW_SPDT
- removed U1: TP4056, meteo_station_footprints:TP4056, symbol meteo_station_symbols:TP4056
- removed U2: LF33_TO220, Package_TO_SOT_THT:TO-220-3_Horizontal_TabDown, symbol meteo_station_symbols:LF33_TO220
- removed U4: DS18B20, meteo_station_footprints:TO-92_Inline, symbol meteo_station_symbols:DS18B20
- removed U5: BH1750, meteo_station_footprints:BH1750, symbol meteo_station_symbols:BH1750
- added J2: PMS7003, Connector:NS-Tech_Grove_1x04_P2mm_Vertical, symbol Connector:Conn_01x04_Pin
- C2: footprint Capacitor_SMD:C_0603_1608Metric -> Capacitor_THT:C_Disc_D7.5mm_W2.5mm_P5.00mm
- R1, R2: footprint Resistor_SMD:R_0603_1608Metric -> Resistor_THT:R_Axial_DIN0207_L6.3mm_D2.5mm_P10.16mm_Horizontal
Connections:
- net OUT+ is gone; now on net 3V3: R1.2
- net OUT- is gone; now on net GND: R2.2
- net GND: now also J2.1 (Pin_1)
- net 5V: now reaches U3.15 (VIN)
- net 5V: now also J2.2 (Pin_2)
- net TX_PMS: now reaches U3.24 (TX2)
- net TX_PMS: now also J2.4 (Pin_4)
- net RX_PMS: now reaches U3.25 (RX2)
- net RX_PMS: now also J2.3 (Pin_3)
- net ADC_BAT: now reaches U3.7 (D33)
- net ADC_BAT: now also C2.1, R1.1, R2.1
- removed net BAT_V: C2.1, R1.1, R2.1, U3.4 (D34)
- no-connect marks 24 -> 20
Other:
- note removed: "OPTIONAL I2C PULL UP"
- moved on the sheet: U3

Commit message: something2
Parts:
- C2: footprint Capacitor_THT:C_Disc_D7.5mm_W2.5mm_P5.00mm -> Capacitor_THT:C_Disc_D5.0mm_W2.5mm_P2.50mm
- J2: footprint Connector:NS-Tech_Grove_1x04_P2mm_Vertical -> Connector_PinHeader_2.54mm:PinHeader_1x04_P2.54mm_Horizontal
Connections:
- net 3V3: no longer C1.1
- net 5V: now also C1.1
Changed lines of the file:
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@@
     )
   )
-  (global_label "3V3" (shape input) (at 29.21 88.9 180) (fields_autoplaced)
-    (effects (font (size 1.27 1.27)) (justify right))
-    (property "Intersheetrefs" "${INTERSHEET_REFS}" (at 23.2893 88.9794 0)
+  (global_label "5V" (shape input) (at 29.21 88.9 180) (fields_autoplaced)
+    (effects (font (size 1.27 1.27)) (justify right))
+    (property "Intersheetrefs" "${INTERSHEET_REFS}" (at 24.0061 88.9 0)
       (effects (font (size 1.27 1.27)) (justify right) hide)
     )
@@
       (effects (font (size 1.27 1.27)) (justify left))
     )
-    (property "Footprint" "Capacitor_THT:C_Disc_D7.5mm_W2.5mm_P5.00mm" (at 56.8452 124.46 0)
+    (property "Footprint" "Capacitor_THT:C_Disc_D5.0mm_W2.5mm_P2.50mm" (at 56.8452 124.46 0)
       (effects (font (size 1.27 1.27)) hide)
     )
@@
       (effects (font (size 1.27 1.27)))
     )
-    (property "Footprint" "Connector:NS-Tech_Grove_1x04_P2mm_Vertical" (at 175.26 63.5 0)
-      (effects (font (size 1.27 1.27)) hide)
-    )
+    (property "Footprint" "Connector_PinHeader_2.54mm:PinHeader_1x04_P2.54mm_Horizontal" (at 175.26 63.5 0)
+      (effects (font (size 1.27 1.27)) hide)
+    )
